File: pcb/cp-vameter.kicad_sch (KiCad schematic)
At the start: 28 parts, among them J1 Vin JST-PH2, J10 Vin Header*, J11 Vin JST-PH2, J12 Grove Ext. INA260, J13 Grove Display, J14 Grove Keypad, J15 Conn Display, J16 Conn Keypad, J2 Vin Header*, J3 Vin Barrel-Jack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

Commit message: replaced tht-footprint with smd-footprint for JST-connector
Parts:
- J1, J11: footprint Connector_JST:JST_PH_S2B-PH-K_1x02_P2.00mm_Horizontal -> Connector_JST:JST_PH_S2B-PH-SM4-TB_1x02-1MP_P2.00mm_Horizontal
Changed lines of the file:
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@@
   (title_block
     (title "cp-vameter")
-    (date "2022-07-05")
-    (rev "1.0")
+    (date "2022-07-29")
+    (rev "1.1")
     (company "Bernhard Bablok")
     (comment 1 "https://github.com/bablokb/circuitpython-vameter")
@@
       (effects (font (size 1.27 1.27)) (justify left))
     )
-    (property "Footprint" "Connector_JST:JST_PH_S2B-PH-K_1x02_P2.00mm_Horizontal" (id 2) (at 133.985 137.16 0)
+    (property "Footprint" "Connector_JST:JST_PH_S2B-PH-SM4-TB_1x02-1MP_P2.00mm_Horizontal" (id 2) (at 133.985 137.16 0)
       (effects (font (size 1.27 1.27)) hide)
     )
@@
       (effects (font (size 1.27 1.27)) (justify left))
     )
-    (property "Footprint" "Connector_JST:JST_PH_S2B-PH-K_1x02_P2.00mm_Horizontal" (id 2) (at 34.925 34.29 0)
+    (property "Footprint" "Connector_JST:JST_PH_S2B-PH-SM4-TB_1x02-1MP_P2.00mm_Horizontal" (id 2) (at 34.925 34.29 0)
       (effects (font (size 1.27 1.27)) hide)
     )
@@
     )
     (path "/fc329e60-968a-4f61-ba77-53d29ff8c1c7"
-      (reference "J1") (unit 1) (value "Vin JST-PH2") (footprint "Connector_JST:JST_PH_S2B-PH-K_1x02_P2.00mm_Horizontal")
+      (reference "J1") (unit 1) (value "Vin JST-PH2") (footprint "Connector_JST:JST_PH_S2B-PH-SM4-TB_1x02-1MP_P2.00mm_Horizontal")
     )
     (path "/03aea3b0-3967-431b-9db8-cf271b1a617d"
@@
     )
     (path "/46883b41-1ec5-4622-b4e3-2cebaa8c855c"
-      (reference "J11") (unit 1) (value "Vin JST-PH2") (footprint "Connector_JST:JST_PH_S2B-PH-K_1x02_P2.00mm_Horizontal")
+      (reference "J11") (unit 1) (value "Vin JST-PH2") (footprint "Connector_JST:JST_PH_S2B-PH-SM4-TB_1x02-1MP_P2.00mm_Horizontal")
     )
     (path "/2683c828-1382-436b-b491-f5c6c9447ffe"
